File: prototype/bbiq_prototype.sch (EAGLE design)
At the start: 17 parts, among them U1 ARDUINOR3-BPLACE, X1 HD44780LCD-1602

Commit message: forgot TMP36
Parts:
- added U2: (no value), SparkFun-Sensors:TMP36GT9
Connections:
- net +5V: now also U2.VCC
- net GND: now also U2.GND
- net TEMP_INTERNAL: now also U2.VOUT
Other:
- moved on the sheet: PROBE_1, PROBE_2, PROBE_3, PROBE_4, R1, R2, R3, R4

Commit message: fixes
Parts:
- added C1: .1uF, rcl:C-US025-025X050
Connections:
- net +5V: now also C1.1
- net GND: now also C1.2
Changed lines of the file:
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@@
 <part name="P+3" library="supply1" library_urn="urn:adsk.eagle:library:371" deviceset="+5V" device=""/>
 <part name="GND7" library="supply1" library_urn="urn:adsk.eagle:library:371" deviceset="GND" device=""/>
+<part name="C1" library="rcl" library_urn="urn:adsk.eagle:library:334" deviceset="C-US" device="025-025X050" package3d_urn="urn:adsk.eagle:package:23629/2" value=".1uF"/>
 </parts>
 <sheets>
@@
 <instance part="P+3" gate="1" x="-15.24" y="-5.08"/>
 <instance part="GND7" gate="1" x="-15.24" y="-20.32"/>
+<instance part="C1" gate="G$1" x="-25.4" y="-12.7"/>
 </instances>
 <busses>
@@
 <wire x1="-15.24" y1="-15.24" x2="-15.24" y2="-17.78" width="0.1524" layer="91"/>
 <pinref part="GND7" gate="1" pin="GND"/>
+<pinref part="C1" gate="G$1" pin="2"/>
+<wire x1="-25.4" y1="-17.78" x2="-15.24" y2="-17.78" width="0.1524" layer="91"/>
+<junction x="-15.24" y="-17.78"/>
 </segment>
 </net>
@@
 <wire x1="-15.24" y1="-10.16" x2="-15.24" y2="-7.62" width="0.1524" layer="91"/>
 <pinref part="P+3" gate="1" pin="+5V"/>
+<pinref part="C1" gate="G$1" pin="1"/>
+<wire x1="-15.24" y1="-10.16" x2="-25.4" y2="-10.16" width="0.1524" layer="91"/>
+<junction x="-15.24" y="-10.16"/>
 </segment>
 </net>
@@
 packages will not be understood (or retained) with this version.
 </note>
+<note version="8.4" severity="warning">
+Since Version 8.4, EAGLE supports properties for SPICE simulation.
+Probes in schematics and SPICE mapping objects found in parts and library devices
+will not be understood with this version. Update EAGLE to the latest version
+for full support of SPICE simulation.
+</note>
 </compatibility>
