File: teensy/BBiQ-1.0.brd (EAGLE design)
At the start: 68.2 x 49.5 mm, 14 parts, among them IC1 ESP-WROOM-02, J1 MJ-2506N, J2 MJ-2506N, J3 MJ-2506N, J4 MJ-2506N

Commit message: schematic
Parts:
- added 0.1µF: (no value), resistor:C025-025X050
- added C1: 10µF, resistor:C025-025X050
- added C2, C3, C4: 0.1µF, resistor:C025-025X050
- added D2: 1N4148DO35-10, diode:DO35-10
- added R1, R2, R3: 10kΩ, resistor:0204/5
- added R4, R5, R6, R7: 10kΩ 1%, resistor:0204/5
- added R8: 1kΩ, resistor:0204/5
- added T1: 2N3904, transistor:TO92
- added U1: (no value), SparkFun-Sensors:TO-92
- S1, S2, S3: value MOMENTARY-SWITCH-SPST-PTH-12MM -> (none)
Connections:
- removed net 3.3V: U$2.3.3V, U$2.3.3V1
- removed net 3V3: IC1.1
- removed net GND0: IC1.19
- removed net GND1: IC1.9
- removed net GND2: IC1.13
- removed net GND3: IC1.18
- new net BUTTON_0: S1.3, U$2.7
- new net BUTTON_1: S2.3, U$2.8
- new net BUTTON_2: S3.3, U$2.9
- new net BUZZER: R3.1, U$2.3
- new net ESP_LOAD: IC1.8, U$2.2
- new net ESP_RST: IC1.15, IC1.17, U$2.12
- new net N$2: C3.1, IC1.2, R1.1
- new net N$3: IC1.6, R2.1
- new net N$4: R3.2, T1.2
- new net N$5: C1.2, C2.2, IC1.1
- new net N$6: D2.A, LS1.-, T1.1
- new net N$7: R8.2, S1.1, S2.1, S3.1
- new net OLED_DC: OLED1.3, U$2.6
- new net OLED_RST: OLED1.2, U$2.4
- new net TMP36: U$2.18/A4, U1.2
- net +3V3: now also 0.1µF.1, C1.1, C2.1, C4.1, D2.C, LS1.+, OLED1.6, R1.2, U$2.3.3V, U$2.3.3V1, U1.1
- net ESP_RX: now also IC1.11
- net ESP_TX: now also IC1.12
- net GND: now also 0.1µF.2, C3.2, C4.2, IC1.13, IC1.18, IC1.19, IC1.9, J1.1, J1.3, J2.1, J2.3, J3.1, J3.3, J4.1, J4.3, R2.2, R8.1, T1.3, U1.3
- net OLED_CK: now also OLED1.4
- net OLED_CS: now also OLED1.1
- net OLED_DATA: now also OLED1.5
- net PROBE0: now also J1.2, R4.1
- net PROBE1: now also J2.2, R5.1
- net PROBE2: now also J3.2, R6.1
- net PROBE3: now also J4.2, R7.1
- net PROBE_PWR: now also R4.2, R5.2, R6.2, R7.2
- net VIN: no longer OLED1.6
