File: teensy/BBiQ-1.0.sch (EAGLE design)
At the start: 14 parts, among them IC1 ESP-WROOM-02, J1 MJ-2506N, J2 MJ-2506N, J3 MJ-2506N, J4 MJ-2506N

Commit message: schematic
Parts:
- added 0.1µF: (no value), resistor:C-US025-025X050
- added C1: 10µF, resistor:C-US025-025X050
- added C2, C3, C4: 0.1µF, resistor:C-US025-025X050
- added D2: 1N4148DO35-10, diode:1N4148DO35-10
- added R1, R2, R3: 10kΩ, resistor:R-US_0204/5
- added R4, R5, R6, R7: 10kΩ 1%, resistor:R-US_0204/5
- added R8: 1kΩ, resistor:R-US_0204/5
- added T1: 2N3904, transistor:2N3904
- added U1: (no value), SparkFun-Sensors:TMP36GT9
Connections:
- new net BUTTON_0: S1.2, U$2.7/RX3
- new net BUTTON_1: S2.2, U$2.8/TX3
- new net BUTTON_2: S3.2, U$2.9/RX2/PWM
- new net BUZZER: R3.1, U$2.3/T/PWM
- new net ESP_LOAD: IC1.IO0, U$2.2
- new net ESP_RST: IC1.IO16, IC1.RST, U$2.12/MISO
- new net N$2: C3.1, IC1.EN, R1.1
- new net N$3: IC1.IO15, R2.1
- new net N$4: R3.2, T1.B
- new net N$5: C1.2, C2.2, IC1.3V3
- new net N$6: D2.A, LS1.2, T1.C
- new net N$7: R8.2, S1.1, S2.1, S3.1
- new net OLED_DC: OLED1.D/C, U$2.6/PWM
- new net OLED_RST: OLED1.RST, U$2.4/T/PWM
- new net TMP36: U$2.18/A4/T/SDA, U1.VOUT
- net +3V3: now also 0.1µF.1, C1.1, C2.1, C4.1, D2.C, LS1.1, OLED1.VIN, R1.2, U$2.3.3V, U1.VCC
- net ESP_RX: now also IC1.RXD
- net ESP_TX: now also IC1.TXD
- net GND: now also 0.1µF.2, C3.2, C4.2, IC1.GND0, IC1.GND1, IC1.GND2, IC1.GND3, J1.1, J1.3, J2.1, J2.3, J3.1, J3.3, J4.1, J4.3, OLED1.GND, R2.2, R8.1, T1.E, U$2.GND, U1.GND
- net OLED_CK: now also OLED1.CLK
- net OLED_CS: now also OLED1.CS
- net OLED_DATA: now also OLED1.DATA
- net PROBE0: now also J1.2, R4.1
- net PROBE1: now also J2.2, R5.1
- net PROBE2: now also J3.2, R6.1
- net PROBE3: now also J4.2, R7.1
- net PROBE_PWR: now also R4.2, R5.2, R6.2, R7.2
Other:
- moved on the sheet: BT1, BT2, IC1, J1, J2, J3, J4, LS1, OLED1, S1, S2, S3
