File: teensy/BBiQ-1.2.sch (EAGLE design)
At the start: 28 parts, among them IC1 ESP-WROOM-02, J1 MJ-2506N, J2 MJ-2506N, J3 MJ-2506N, J4 MJ-2506N, T1 2N3904

Commit message: tweaks
Parts:
- added C6: 1000µF, resistor:CPOL-USE3.5-8
- added U$3, U$4, U$5, U$6: MOUNTINGHOLE2.5, microbuilder:MOUNTINGHOLE2.5
- C4: device resistor:C-US025-025X050 -> resistor:CPOL-USE2-5
Connections:
- net +3V3: now also C4.+, C6.+; no longer C4.1
- net GND: now also C4.-, C6.-; no longer C4.2
Changed lines of the file:
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@@
 <part name="GND7" library="supply1" library_urn="urn:adsk.eagle:library:371" deviceset="GND" device=""/>
 <part name="C3" library="resistor" library_urn="urn:adsk.eagle:library:348" deviceset="C-US" device="025-025X050" package3d_urn="urn:adsk.eagle:package:23629/2" value="0.1µF"/>
-<part name="C4" library="resistor" library_urn="urn:adsk.eagle:library:348" deviceset="C-US" device="025-025X050" package3d_urn="urn:adsk.eagle:package:23629/2" value="10µF"/>
 <part name="+3V2" library="supply1" library_urn="urn:adsk.eagle:library:371" deviceset="+3V3" device=""/>
 <part name="C5" library="resistor" library_urn="urn:adsk.eagle:library:348" deviceset="C-US" device="025-025X050" package3d_urn="urn:adsk.eagle:package:23629/2" value="0.1µF"/>
@@
 <part name="R8" library="resistor" library_urn="urn:adsk.eagle:library:348" deviceset="R-US_" device="0207/7" package3d_urn="urn:adsk.eagle:package:23493/1" value="10k 1%"/>
 <part name="GND9" library="supply1" library_urn="urn:adsk.eagle:library:371" deviceset="GND" device=""/>
+<part name="U$3" library="microbuilder" deviceset="MOUNTINGHOLE" device="2.5"/>
+<part name="U$4" library="microbuilder" deviceset="MOUNTINGHOLE" device="2.5"/>
+<part name="U$5" library="microbuilder" deviceset="MOUNTINGHOLE" device="2.5"/>
+<part name="U$6" library="microbuilder" deviceset="MOUNTINGHOLE" device="2.5"/>
+<part name="C4" library="resistor" library_urn="urn:adsk.eagle:library:348" deviceset="CPOL-US" device="E2-5" package3d_urn="urn:adsk.eagle:package:23346/2" value="10µF"/>
+<part name="C6" library="resistor" library_urn="urn:adsk.eagle:library:348" deviceset="CPOL-US" device="E3.5-8" package3d_urn="urn:adsk.eagle:package:23360/2" value="1000µF"/>
 </parts>
 <sheets>
@@
 <instance part="GND7" gate="1" x="144.78" y="45.72"/>
 <instance part="C3" gate="G$1" x="129.54" y="134.62" rot="R90"/>
-<instance part="C4" gate="G$1" x="129.54" y="142.24" rot="R90"/>
-<instance part="+3V2" gate="G$1" x="127" y="152.4"/>
+<instance part="+3V2" gate="G$1" x="127" y="160.02"/>
 <instance part="C5" gate="G$1" x="129.54" y="124.46" rot="R90"/>
 <instance part="R5" gate="G$1" x="127" y="129.54" rot="R90"/>
@@
 <instance part="R8" gate="G$1" x="5.08" y="91.44" rot="R90"/>
 <instance part="GND9" gate="1" x="5.08" y="83.82"/>
+<instance part="U$3" gate="G$1" x="-35.56" y="91.44"/>
+<instance part="U$4" gate="G$1" x="-35.56" y="83.82"/>
+<instance part="U$5" gate="G$1" x="-35.56" y="76.2"/>
+<instance part="U$6" gate="G$1" x="-35.56" y="68.58"/>
+<instance part="C4" gate="G$1" x="129.54" y="142.24" rot="R90"/>
+<instance part="C6" gate="G$1" x="129.54" y="149.86" rot="R90"/>
 </instances>
 <busses>
@@
 <pinref part="IC1" gate="G$1" pin="GND0"/>
 <junction x="124.46" y="106.68"/>
-<pinref part="C4" gate="G$1" pin="2"/>
 <pinref part="C3" gate="G$1" pin="2"/>
 <wire x1="134.62" y1="142.24" x2="134.62" y2="134.62" width="0.1524" layer="91"/>
@@
 <pinref part="R6" gate="G$1" pin="2"/>
 <junction x="134.62" y="114.3"/>
+<pinref part="C4" gate="G$1" pin="-"/>
+<pinref part="C6" gate="G$1" pin="-"/>
+<wire x1="134.62" y1="149.86" x2="134.62" y2="142.24" width="0.1524" layer="91"/>
+<junction x="134.62" y="142.24"/>
 </segment>
 <segment>
@@
 <wire x1="124.46" y1="134.62" x2="127" y2="134.62" width="0.1524" layer="91"/>
 <pinref part="+3V2" gate="G$1" pin="+3V3"/>
-<pinref part="C4" gate="G$1" pin="1"/>
-<junction x="127" y="142.24"/>
 <wire x1="127" y1="134.62" x2="127" y2="142.24" width="0.1524" layer="91"/>
 <wire x1="127" y1="142.24" x2="127" y2="149.86" width="0.1524" layer="91"/>
@@
 <junction x="127" y="134.62"/>
 <pinref part="R5" gate="G$1" pin="2"/>
+<pinref part="C4" gate="G$1" pin="+"/>
+<junction x="127" y="142.24"/>
+<pinref part="C6" gate="G$1" pin="+"/>
+<wire x1="127" y1="149.86" x2="127" y2="157.48" width="0.1524" layer="91"/>
+<junction x="127" y="149.86"/>
 </segment>
 <segment>
@@
 </sheet>
 </sheets>
+<errors>
+</errors>
 </schematic>
 </drawing>
